File: bots/flipping-cool/pcb/00_system_overview.kicad_sch (KiCad schematic)
At the start: 0 parts

Commit message: Refactor Flipping Cool PCB design to Rev B, updating title, date, and revision details. Integrate ESP32-S3 module and enhance documentation for MCU I/O and debugging features, while maintaining historical context from Rev A.
Other:
- note added: "Critical safety wiring: MODE_SAFE/MODE_RX_DIRECT/MODE_MCU_CONTROL each have 100k pull-downs, so undefined switch travel cannot float authority nets."
- note added: "Flipping Cool Rev B single-board integrated control/power design"
- note added: "MCU_CONTROL: MODE_MCU_CONTROL high. SERVO_6V_SW enabled. PWM mux select switches to ESP32-S3 outputs. BLE/firmware authority only in this state."
- note added: "Off-board boundary (intentional): 2S battery pack, WEKA dual brushed ESC, 4 drive motors, 2 weapon servos, Matek ELRS-R24-P6 receiver."
- note added: "Power tree: J1 battery -> J2 removable link -> VBAT_SW. VBAT_SW feeds U20 6V servo buck, U21 RX_5V regulator, U30 AUX_3V3 buck, D1 TVS, C1/C2 bulk, and test points."
- note added: "RX_DIRECT: MODE_RX_DIRECT high. SERVO_6V_SW enabled. PWM mux select forced to receiver channel inputs. Works with MCU absent or crashed."
- note added: "Rail naming contract: VBAT_RAW before disconnect, VBAT_SW after link, SERVO_6V from U20, SERVO_6V_SW after Q1, RX_5V from U21, AUX_3V3 from U30, GND_PWR common return."
- note added: "Receiver-priority authority model (hardware-enforced):"
- note added: "Rev B implementation rule: this schematic is authoritative. PCB must stay synchronized from this source before any routing or fab release."
- note added: "SAFE: MODE_SAFE high, MODE_RX_DIRECT low, MODE_MCU_CONTROL low. SERVO_6V_SW disabled through Q1 load switch. PWM mux defaults to receiver side while servo rail is cut."
- note added: "Validated source set: Pololu 3064 motors, Savox SH-0255MG+, GNB 2S LiHV 450mAh pack, Matek ELRS-R24-P6, WEKA dual brushed ESC, Pololu D36V50F6."
- note removed: "Architecture: 2S LiHV XT30 battery -> manual removable link -> VBAT_SW -> WEKA drive ESC and Pololu D36V50F6 6V BEC. ELRS PWM receiver drives WEKA and two Savox weapon servos. No custom ESC, no required MCU. Optional growth hooks add pit/debug, 3.3V sensor/MCU power, I2C, ADC rail sense, and RGB status LED support."
- note removed: "Flipping Cool Rev A schematic-only power/interconnect PCB"
- note removed: "Growth constraints: optional MCU/PWM points are passive taps in Rev A; they must not drive receiver-owned PWM nets unless the harness is intentionally reworked. AUX_3V3 is switched off by the main link through VBAT_SW."
- note removed: "Load budget: drive motors 4 x 1.5A stall at 6V = 6A nominal stall reference; weapon servos 2 x 1.4A stall at 6V = 2.8A; BEC target >=4A real headroom, implemented as 6V 5.5A module. 2S directly overvolts 6V motors, so stall duration must be mechanically and operationally limited."
- note removed: "Rail names: VBAT_RAW = battery side of disconnect; VBAT_SW = robot-live switched battery rail; SERVO_6V = external 6V BEC output; RX_6V = filtered receiver branch; AUX_3V3 = optional future logic/sensor rail; GND_PWR = common return."
- note removed: "Safety requirements captured here: mechanical main battery disconnect, visible power indication tied to VBAT_SW, protected battery terminals, and receiver/servo rail isolated from the WEKA logic-only BEC."
- note removed: "Validated remote sources: Pololu 3064 motor specs https://www.pololu.com/product/3064/specs ; Savox SH-0255MG+ specs https://www.teamsavox.com/product/sh-0255mgp/ ; GNB4502S80AHV https://www.gaoneng.shop/products/gaoneng-gnb-lihv-2s-7-6v-450mah-80c-xt30-lipo-battery ; SPARC v1.6 https://www.sparc.tools/SPARC_Robot_Construction_Specifications_v1.6.pdf ; Matek ELRS-R24-P6 https://www.mateksys.com/?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"
- title: Flipping Cool Rev A - System Overview -> Flipping Cool Rev B - System Overview
Changed lines of the file:
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@@
   (paper "A4")
   (title_block
-    (title "Flipping Cool Rev A - System Overview")
-    (date "2026-05-08")
-    (rev "A")
+    (title "Flipping Cool Rev B - System Overview")
+    (date "2026-05-09")
+    (rev "B")
     (company "battle_bots_ai")
   )
-  (text "Flipping Cool Rev A schematic-only power/interconnect PCB"
-    (at 15.00 18.00 0)
+  (text "Flipping Cool Rev B single-board integrated control/power design"
+    (at 15.00 16.00 0)
     (effects (font (size 1.80 1.80)) (justify left top))
   )
-  (text "Architecture: 2S LiHV XT30 battery -> manual removable link -> VBAT_SW -> WEKA drive ESC and Pololu D36V50F6 6V BEC. ELRS PWM receiver drives WEKA and two Savox weapon servos. No custom ESC, no required MCU. Optional growth hooks add pit/debug, 3.3V sensor/MCU power, I2C, ADC rail sense, and RGB status LED support."
-    (at 15.00 26.00 0)
+  (text "Off-board boundary (intentional): 2S battery pack, WEKA dual brushed ESC, 4 drive motors, 2 weapon servos, Matek ELRS-R24-P6 receiver."
+    (at 15.00 24.00 0)
     (effects (font (size 1.27 1.27)) (justify left top))
   )
-  (text "Rail names: VBAT_RAW = battery side of disconnect; VBAT_SW = robot-live switched battery rail; SERVO_6V = external 6V BEC output; RX_6V = filtered receiver branch; AUX_3V3 = optional future logic/sensor rail; GND_PWR = common return."
-    (at 15.00 38.00 0)
+  (text "Power tree: J1 battery -> J2 removable link -> VBAT_SW. VBAT_SW feeds U20 6V servo buck, U21 RX_5V regulator, U30 AUX_3V3 buck, D1 TVS, C1/C2 bulk, and test points."
+    (at 15.00 34.00 0)
     (effects (font (size 1.27 1.27)) (justify left top))
   )
-  (text "Load budget: drive motors 4 x 1.5A stall at 6V = 6A nominal stall reference; weapon servos 2 x 1.4A stall at 6V = 2.8A; BEC target >=4A real headroom, implemented as 6V 5.5A module. 2S directly overvolts 6V motors, so stall duration must be mechanically and operationally limited."
-    (at 15.00 52.00 0)
-    (effects (font (size 1.27 1.27)) (justify left top))
+  (text "Receiver-priority authority model (hardware-enforced):"
+    (at 15.00 45.00 0)
+    (effects (font (size 1.27 1.27) bold yes) (justify left top))
   )
-  (text "Validated remote sources: Pololu 3064 motor specs https://www.pololu.com/product/3064/specs ; Savox SH-0255MG+ specs https://www.teamsavox.com/product/sh-0255mgp/ ; GNB4502S80AHV https://www.gaoneng.shop/products/gaoneng-gnb-lihv-2s-7-6v-450mah-80c-xt30-lipo-battery ; SPARC v1.6 https://www.sparc.tools/SPARC_Robot_Construction_Specifications_v1.6.pdf ; Matek ELRS-R24-P6 https://www.mateksys.com/?portfolio=elrs-r24-p6 ; WEKA ESC https://justcuzrobotics.com/products/weka-dual-20-esc-for-brushed-drive ; Pololu D36V50F6 https://www.pololu.com/product/4092 ; Pololu D24V5F3 https://www.pololu.com/product/2842 ; STEMMA QT pin order https://learn.adafruit.com/introducing-adafruit-stemma-qt/technical-specs"
-    (at 15.00 73.00 0)
+  (text "SAFE: MODE_SAFE high, MODE_RX_DIRECT low, MODE_MCU_CONTROL low. SERVO_6V_SW disabled through Q1 load switch. PWM mux defaults to receiver side while servo rail is cut."
+    (at 15.00 51.00 0)
     (effects (font (size 1.05 1.05)) (justify left top))
   )
-  (text "Safety requirements captured here: mechanical main battery disconnect, visible power indication tied to VBAT_SW, protected battery terminals, and receiver/servo rail isolated from the WEKA logic-only BEC."
-    (at 15.00 108.00 0)
-    (effects (font (size 1.27 1.27)) (justify left top))
+  (text "RX_DIRECT: MODE_RX_DIRECT high. SERVO_6V_SW enabled. PWM mux select forced to receiver channel inputs. Works with MCU absent or crashed."
+    (at 15.00 59.00 0)
+    (effects (font (size 1.05 1.05)) (justify left top))
   )
-  (text "Growth constraints: optional MCU/PWM points are passive taps in Rev A; they must not drive receiver-owned PWM nets unless the harness is intentionally reworked. AUX_3V3 is switched off by the main link through VBAT_SW."
-    (at 15.00 120.00 0)
-    (effects (font (size 1.27 1.27)) (justify left top))
+  (text "MCU_CONTROL: MODE_MCU_CONTROL high. SERVO_6V_SW enabled. PWM mux select switches to ESP32-S3 outputs. BLE/firmware authority only in this state."
+    (at 15.00 67.00 0)
+    (effects (font (size 1.05 1.05)) (justify left top))
+  )
+  (text "Critical safety wiring: MODE_SAFE/MODE_RX_DIRECT/MODE_MCU_CONTROL each have 100k pull-downs, so undefined switch travel cannot float authority nets."
+    (at 15.00 75.00 0)
+    (effects (font (size 1.05 1.05)) (justify left top))
+  )
+  (text "Rail naming contract: VBAT_RAW before disconnect, VBAT_SW after link, SERVO_6V from U20, SERVO_6V_SW after Q1, RX_5V from U21, AUX_3V3 from U30, GND_PWR common return."
+    (at 15.00 84.00 0)
+    (effects (font (size 1.05 1.05)) (justify left top))
+  )
+  (text "Validated source set: Pololu 3064 motors, Savox SH-0255MG+, GNB 2S LiHV 450mAh pack, Matek ELRS-R24-P6, WEKA dual brushed ESC, Pololu D36V50F6."
+    (at 15.00 95.00 0)
+    (effects (font (size 1.00 1.00)) (justify left top))
+  )
+  (text "Rev B implementation rule: this schematic is authoritative. PCB must stay synchronized from this source before any routing or fab release."
+    (at 15.00 104.00 0)
+    (effects (font (size 1.05 1.05) bold yes) (justify left top))
   )
   (sheet_instances
