File: bots/flipping-cool/pcb/06_expansion_test.kicad_sch (KiCad schematic)
At the start: 38 parts, among them J40 SPARE_SWITCHED_VBAT_OUT_FUSED, J41 SPARE_6V_ACCESSORY, J42 OPTIONAL_CRSF_UART_PADS, J43 PWM_SPARE_BREAKOUT, J44 PIT_DEBUG_POWER_COMMS, J45 OPTIONAL_POLOLU_D24V5F3_3V3, J46 FUTURE_MCU_POWER_COMMS, J47 FUTURE_MCU_PWM_I2C_TAPS, J48 FUTURE_MCU_ADC_LED, J49 I2C_SENSOR_STEMMA_QT_QWIIC, J50 COMMON_ANODE_RGB_STATUS_LED

Commit message: Refactor Flipping Cool PCB design to Rev B, updating title, date, and revision details. Integrate ESP32-S3 module and enhance documentation for MCU I/O and debugging features, while maintaining historical context from Rev A.
Parts:
- added C10: 1uF_EN_CAP, Capacitor_SMD:C_0805_2012Metric, symbol Device:C
- added J12: UART_PROGRAM_HEADER, Connector_PinHeader_2.54mm:PinHeader_1x06_P2.54mm_Vertical, symbol Connector_Generic:Conn_01x06
- added J13: USB_DEBUG_BREAKOUT, Connector_USB:USB_C_Receptacle_GCT_USB4085, symbol Connector_Generic:Conn_01x04
- added R10: 10k_EN_PULLUP, Resistor_SMD:R_0805_2012Metric, symbol Device:R
- added R11: 10k_BOOT_PULLUP, Resistor_SMD:R_0805_2012Metric, symbol Device:R
- added SW2: RESET_BTN, Button_Switch_SMD:SW_SPST_TL3305B, symbol Connector_Generic:Conn_01x02
- added SW3: BOOT_BTN, Button_Switch_SMD:SW_SPST_TL3305B, symbol Connector_Generic:Conn_01x02
- added U10: ESP32-S3-WROOM-1, RF_Module:ESP32-S3-WROOM-1, symbol custom:ESP32_S3_WROOM_1_WRAPPER
- added U11: USBLC6-2SC6, Package_TO_SOT_SMD:SOT-23-6, symbol custom:ESD_USBLC6_2SC6
Connections:
- net ADC_RX_6V: now also U10.7 (IO7)
- net ADC_SERVO_6V: now also U10.12 (IO8)
- net ADC_VBAT: now also U10.13 (IO9)
- net AUX_3V3: now also R10.2, R11.2, U10.20 (USB_D+)
- net GND_PWR: now also J13.4 (Pin_4), SW2.2 (Pin_2), SW3.2 (Pin_2), U11.3 (I/O2)
- net I2C_SCL: now also U10.39 (IO1_ADC)
- net I2C_SDA: now also U10.40 (IO2_ADC)
- net STATUS_LED_B_N: now also U10.16 (IO12)
- net STATUS_LED_G_N: now also U10.17 (IO13)
- net STATUS_LED_R_N: now also U10.18 (IO14)
- new net ESP_BOOT: R11.1, SW3.1 (Pin_1), U10.6 (IO6)
- new net ESP_EN: R10.1, SW2.1 (Pin_1), U10.19 (USB_D-)
- new net MCU_PWM_DRIVE_LEFT: U10.38 (U0RXD)
- new net MCU_PWM_DRIVE_RIGHT: U10.37 (U0TXD)
- new net MCU_PWM_WEAPON_FR: U10.27 (IO0_BOOT)
- new net MCU_PWM_WEAPON_LR: U10.41 (IO3_ADC)
- new net UART0_RXD: U10.4 (IO4)
- new net UART0_TXD: U10.5 (IO5)
- new net USB_CONN_D_N: J13.2 (Pin_2), U11.5 (VBUS)
- new net USB_CONN_D_P: J13.1 (Pin_1)
- new net USB_D_N: U10.3 (EN)
- new net USB_D_P: U10.2 (3V3), U11.2 (GND)
- new net VBUS_5V_USB: J13.3 (Pin_3)
Other:
- note added: "U10 pin map uses Rev B wrapper: IO0 boot strap on ESP_BOOT, UART0 on J12, native USB on IO19/IO20, rail ADC on IO1/IO2/IO3."
- title: Flipping Cool Rev A - Expansion and Test -> Flipping Cool Rev B - MCU IO and Debug
